File: KiCAD/PowerSupply.sch (KiCad schematic (older format))
At the start: 12 parts, among them J4 USB-Micro, Q1 3.7A, 30V, U2 LM1117, U3 AP2112K-3.3

Commit message: Fix library error
Parts:
- U2: symbol LM1117 -> LM1117-RESCUE-SAMD21-DevBoard
Other:
- note removed: "VERIFY USB PINOUT"
Changed lines of the file:
@@
 EESchema Schematic File Version 2
+LIBS:SAMD21-DevBoard-rescue
 LIBS:power
 LIBS:device
@@
 	7250 3450 7750 3450
 $Comp
-L LM1117 U2
+L LM1117-RESCUE-SAMD21-DevBoard U2
 U 1 1 5C0C6154
 P 5900 4850
+AR Path="/5C0C6154" Ref="U2"  Part="1"
+AR Path="/5BF26B92/5C0C6154" Ref="U2"  Part="1"
 F 0 "U2" H 5750 4975 50  0000 C CNN
 F 1 "LM1117" H 5900 4975 50  0000 L CNN
@@
 	6250 4950 6250 4850
 Connection ~ 6250 4850
-Text Notes 3250 2900 0    79   ~ 0
-VERIFY USB PINOUT
 NoConn ~ 4450 3750
 $EndSCHEMATC
